Commit message: Update DH116S left and right hand model files
Update STL meshes, MJCF XML configs, URDF files, and simulation scripts
for both DH116S-L000-A1 and DH116S-R000-A1 hand models.

Co-Authored-By: Claude Opus 4.7 <noreply@anthropic.com>

File: DH116S/DH116S_URDF_MJCF_Files/DH116S-L000-A1/urdf/DH116S-L000-A1.urdf (robot description, URDF)
Before this commit: robot DH116S-L000-A1, 17 links, 16 joints
Links:
- link base_link: mass 0.10796 -> 0.106661851888605
- link finger11_link: mass 0.0027298 -> 0.00703896093413542
- link finger12_link: mass 0.15692 -> 0.00572071000157471
- link finger13_link: mass 0.0051235 -> 0.00512347195060515
- link finger14_link: mass 0.0024051 -> 0.00240509776372723
- link finger21_link: mass 0.003938 -> 0.00393802264883532
- link finger22_link: mass 0.0035951 -> 0.00359512240318104
- link finger23_link: mass 0.0019493 -> 0.00194918551000528
- link finger31_link: mass 0.0046564 -> 0.00465629805037929
- link finger32_link: mass 0.0039652 -> 0.00396494093318317
- link finger33_link: mass 0.0022728 -> 0.00227281439382211
- link finger41_link: mass 0.0041427 -> 0.00414279060803409
- link finger42_link: mass 0.0038285 -> 0.00382854887772676
- link finger43_link: mass 0.0019493 -> 0.00194917712642498
- link finger51_link: mass 0.0034504 -> 0.00345036527036827
- link finger52_link: mass 0.0034586 -> 0.00345865291103541
- link finger53_link: mass 0.0014962 -> 0.00149700207994512
Joints:
- joint finger11: limit lower=0 upper=1.75 effort=0 velocity=0 -> lower=0 upper=1.588 effort=0 velocity=0; origin xyz=0.019352 0.0078052 0.03432 rpy=0 5.6618E-05 0 -> xyz=0.0193521365394396 0.00780520239676655 0.0343200230340877 rpy=0 5.66182786981891E-05 0
- joint finger12: limit lower=0 upper=1.40 effort=0 velocity=0 -> lower=0 upper=1.030 effort=0 velocity=0; origin xyz=0.015 0.0024172 0.0067143 rpy=1.1789 0.2618 1.5708 -> xyz=0.0149999999999999 0.00241716818236522 0.00671430739572605 rpy=0.914542570706424 0.26179938779915 1.5707963267949
- joint finger13: mimic joint=finger12 multiplier=0.929 offset=-0.015082 -> joint=finger12 multiplier=0.88178789 offset=-0.00697725445; origin xyz=0 0 0.040273 rpy=0 0 0 -> xyz=0.000907073874635978 -0.012631430230703 0.0382111085733653 rpy=0.320192464474519 0.0133797340704482 0.0102567262059099
- joint finger21: limit lower=0 upper=1.40 effort=0 velocity=0 -> lower=0 upper=1.257 effort=0 velocity=0; origin xyz=0.026322 -0.0053264 0.083909 rpy=0.015713 0.09766 0.15979 -> xyz=0.0263221667373393 -0.00532638133131497 0.0839088174238425 rpy=0.0157127180588976 0.0976603903613511 0.159786795598776
- joint finger22: mimic joint=finger21 multiplier=0.8847 offset=0.038265 -> joint=finger21 multiplier=1.36723967 offset=-0.0628270617; origin xyz=0 0.0030778 0.027857 rpy=-0.11004 0 0 -> xyz=0 0.00510326179486572 0.027558142915563 rpy=-0.183107378899691 0 0
- joint finger31: limit lower=0 upper=1.40 effort=0 velocity=0 -> lower=0 upper=1.257 effort=0 velocity=0; origin xyz=0.0085306 -0.006534 0.088185 rpy=0.00071294 0.013408 0.053126 -> xyz=0.00853056012195752 -0.00653399721710813 0.08818546795159 rpy=0.000712944465730327 0.0134076578043506 0.0531259881623533
- joint finger32: mimic joint=finger31 multiplier=0.8485 offset=0.035946 -> joint=finger31 multiplier=1.39585814 offset=-0.0787255295; origin xyz=0 0.0037175 0.032318 rpy=0 0 0 -> xyz=0 0.00597179476535116 0.031978135864213 rpy=0 0 0
- joint finger41: limit lower=0 upper=1.40 effort=0 velocity=0 -> lower=0 upper=1.257 effort=0 velocity=0; origin xyz=-0.0088876 -0.0072813 0.087396 rpy=0.0030266 -0.061554 -0.049162 -> xyz=-0.00888762654492145 -0.00728133879903732 0.087396405615583 rpy=0.00302662499820262 -0.0615538222955632 -0.0491619519178472
- joint finger42: mimic joint=finger41 multiplier=0.8321 offset=0.043170 -> joint=finger41 multiplier=1.40106471 offset=-0.0760281065; origin xyz=0 0.0025283 0.02942 rpy=0 0 0 -> xyz=0 0.0054849861571379 0.0290146270636347 rpy=0 0 0
- joint finger51: limit lower=0 upper=1.40 effort=0 velocity=0 -> lower=0 upper=1.291 effort=0 velocity=0; origin xyz=-0.026448 -0.0055489 0.08298 rpy=-0.074855 -0.15057 -0.14704 -> xyz=-0.0264481824708094 -0.0055488670962835 0.0829799586736383 rpy=-0.153756050317575 -0.150571871776981 -0.147041448694914
- joint finger52: mimic joint=finger51 multiplier=0.7349 offset=0.035218 -> joint=finger51 multiplier=1.28966594 offset=-0.0841491377; origin xyz=0 0 0.025024 rpy=0.097068 0 0 -> xyz=0 0 0.0250241718362191 rpy=0.175969487717828 0 0

File: DH116S/DH116S_URDF_MJCF_Files/DH116S-R000-A1/urdf/DH116S-R000-A1.urdf (robot description, URDF)
Before this commit: robot DH116S-R000-A1, 17 links, 16 joints
Links:
- link base_link: mass 0.10795 -> 0.109379461925353
- link finger11_link: mass 0.0027298 -> 0.00704884300354655
- link finger12_link: mass 0.15691 -> 0.00572064501582461
- link finger13_link: mass 0.0051235 -> 0.00512347606012059
- link finger14_link: mass 0.0024048 -> 0.00240482348656883
- link finger21_link: mass 0.0039377 -> 0.00393774528740839
- link finger22_link: mass 0.0035951 -> 0.00359509305446838
- link finger23_link: mass 0.0019493 -> 0.00194916130998001
- link finger31_link: mass 0.0046564 -> 0.00465632374460654
- link finger32_link: mass 0.0039648 -> 0.00396485659955852
- link finger33_link: mass 0.0022727 -> 0.00227280089263279
- link finger41_link: mass 0.0041427 -> 0.0041427825906401
- link finger42_link: mass 0.0038285 -> 0.00382855237153465
- link finger43_link: mass 0.0019493 -> 0.00194917989840034
- link finger51_link: mass 0.0034504 -> 0.00345037170327943
- link finger52_link: mass 0.0034587 -> 0.0034586827978682
- link finger53_link: mass 0.0014968 -> 0.00149578721592064
Joints:
- joint finger11: limit lower=0 upper=1.75 effort=0 velocity=0 -> lower=0 upper=1.588 effort=0 velocity=0; origin xyz=0.019011 -0.007805 0.03432 rpy=0 -3.0438E-05 1.5708 -> xyz=0.019011443942029 -0.00780399999999971 0.0343199999999998 rpy=0 0 1.4189526818714
- joint finger12: limit lower=0 upper=1.40 effort=0 velocity=0 -> lower=0 upper=1.030 effort=0 velocity=0; origin xyz=-0.0024172 -0.015 0.0067143 rpy=1.1997 -0.2618 0 -> xyz=-0.00241716818193387 -0.0149999999957004 0.00671430739411609 rpy=0.914460600969039 -0.26179938779915 0
- joint finger13: mimic joint=finger12 multiplier=0.929 offset=-0.015082 -> joint=finger12 multiplier=0.88178789 offset=-0.00697725445; origin xyz=0 0 0.040273 rpy=0 0 0 -> xyz=0.00598654106733671 -0.0125165261747051 0.0381626484720598 rpy=0.382919042912385 0.147573481949468 0.0154304498115495
- joint finger21: limit lower=0 upper=1.40 effort=0 velocity=0 -> lower=0 upper=1.257 effort=0 velocity=0; origin xyz=0.026269 0.0052799 0.083877 rpy=-0.018831 0.11816 -0.15867 -> xyz=0.0262687686016299 0.00528244145664834 0.0838772330726273 rpy=0.184030828348921 0.0900710961718212 0
- joint finger22: mimic joint=finger21 multiplier=0.8847 offset=0.038265 -> joint=finger21 multiplier=1.36723967 offset=-0.0628270617; origin xyz=0 -0.0036408 0.027789 rpy=0 0 0 -> xyz=0 0 0.028026675184573 rpy=0 0 0
- joint finger31: limit lower=0 upper=1.40 effort=0 velocity=0 -> lower=0 upper=1.257 effort=0 velocity=0; origin xyz=0.008744 0.006507 0.088166 rpy=0.10576 0.052052 -0.049525 -> xyz=0.00874401205559361 0.00650966935499851 0.0881661201014335 rpy=0.175821944347936 0.05205044550937 -0.0495268334341439
- joint finger32: mimic joint=finger31 multiplier=0.8485 offset=0.035946 -> joint=finger31 multiplier=1.39585814 offset=-0.0787255295; origin xyz=0 -0.00026526 0.03253 rpy=0 0 0 -> xyz=0 -0.000265259842373017 0.0325298807757662 rpy=0 0 0
- joint finger41: limit lower=0 upper=1.40 effort=0 velocity=0 -> lower=0 upper=1.257 effort=0 velocity=0; origin xyz=-0.0088463 0.0073041 0.087413 rpy=0.082606 -0.034779 0.050937 -> xyz=-0.00884629646917347 0.007306751562741 0.0874130612220856 rpy=0.185216698200614 -0.0252760066009568 0
- joint finger42: mimic joint=finger41 multiplier=0.8321 offset=0.043170 -> joint=finger41 multiplier=1.40106471 offset=-0.0760281065; origin xyz=0 0 0.029529 rpy=-0.084349 0 0 -> xyz=0 0 0.0295285227667386 rpy=0 0 0
- joint finger51: limit lower=0 upper=1.40 effort=0 velocity=0 -> lower=0 upper=1.291 effort=0 velocity=0; origin xyz=-0.026313 0.0056254 0.083042 rpy=0.076915 -0.11667 0.14928 -> xyz=-0.0263133099109462 0.00562794981638235 0.0830420444966198 rpy=0.153405557961376 -0.116668550344774 0.149285285649185
- joint finger52: mimic joint=finger51 multiplier=0.7349 offset=0.035218 -> joint=finger51 multiplier=1.28966594 offset=-0.0841491377; origin xyz=0 0 0.025024 rpy=0 0 0 -> xyz=0 0 0.0250241718362191 rpy=0 0 0
