Commit message: DH116: refresh L/R hands from the new CAD export
Replace the hand-maintained parts of both DH116 packages with the output of
the new SolidWorks export, re-applying the manual work through scripts:

- tools/patch_sw2urdf_limits.py: mimic couplings, joint travel limits
  (57/43/63/63/62/66 deg), fingertip colours, fixed-joint axes, link/mesh
  name normalisation and line endings.  The linear URDF mimic is now fitted
  as the chord of the quadratic over the travel range (exact at both ends,
  max 3.8 deg mid-range) instead of the first-order term, which used to lag
  14-15 deg at full travel compared with the MJCF polycoef.
- tools/urdf2mjcf.py: MJCF is generated from the URDF, so body poses,
  ranges, inertials, colours and the quadratic equality all come from one
  source.  sim_hand.py is shared by both hands and resolves its model file
  automatically.
- Left hand: link and mesh names normalised to lowercase *_link, thumb zero
  updated by -25.34 deg about finger11 to match the new CAD, base mass from
  the new thumb mount part.

Also drop the tracked export.log files from DH116V2.0, ignore
export.log/.DS_Store/__pycache__, and update the README tables (limits,
mimic) plus the post-export workflow.

File: DH116/DH116_URDF_MJCF_Files/DH116-L000-A1/urdf/DH116-L000-A1.urdf (robot description, URDF)
Before this commit: robot DH116-L000-A1, 17 links, 16 joints
Links:
- link base_link: mass 0.11674 -> 0.182082775508813
- link finger11_link: mass 0.010254 -> 0.0100354213148386
- link finger12_link: mass 0.010117 -> 0.0101165351943037
- link finger13_link: mass 0.020548 -> 0.0205475839130716
- link finger14_link: mass 0.00063385 -> 0.00063385693690849
- link finger21_link: mass 0.0067138 -> 0.00671369658320003
- link finger22_link: mass 0.014791 -> 0.0147901748535033
- link finger23_link: mass 0.00081811 -> 0.000818165979185504
- link finger31_link: mass 0.0067137 -> 0.00671382886294791
- link finger32_link: mass 0.017437 -> 0.0174354297727344
- link finger33_link: mass 0.00081807 -> 0.000818142292598219
- link finger41_link: mass 0.0067137 -> 0.0067137191686616
- link finger42_link: mass 0.014791 -> 0.0147900078598475
- link finger43_link: mass 0.00081812 -> 0.000818155456735261
- link finger51_link: mass 0.0067139 -> 0.00671392149187143
- link finger52_link: mass 0.010439 -> 0.0104389557015327
- link finger53_link: mass 0.00058044 -> 0.00058047721345209
Joints:
- joint finger11: axis 0 0 1 -> 0 -1 0; limit lower=0 upper=1.047198 effort=0 velocity=0 -> lower=0.000000 upper=0.994838 effort=0 velocity=0; origin xyz=0.018 -0.021464 0.040041 rpy=0.087266 0 0 -> xyz=0.018 -0.021721 0.04198 rpy=-1.5708 0.066815 -2.2708
- joint finger12: limit lower=0 upper=0.523599 effort=0 velocity=0 -> lower=0.000000 upper=0.750492 effort=0 velocity=0; origin xyz=0.018876 -0.0049375 -0.0023593 rpy=0 0.95149 -0.25585 -> xyz=0 0.0069955 0.019148 rpy=0 -0.56313 1.5708
- joint finger13: limit lower=0.004592 upper=0.594583 effort=0 velocity=0 -> lower=0.004592 upper=0.930248 effort=0 velocity=0; mimic joint=finger12 multiplier=0.8808 offset=0.004592 -> joint=finger12 multiplier=1.233400 offset=0.004592
- joint finger14: limit lower=0 upper=1.396263 effort=0 velocity=0 -> lower=0 upper=1.57 effort=0 velocity=0
- joint finger21: limit lower=0 upper=1.396263 effort=0 velocity=0 -> lower=0.000000 upper=1.099557 effort=0 velocity=0; origin xyz=-0.011581 -0.031971 0.10003 rpy=0.052657 0.10625 0.0055894 -> xyz=-0.011581 -0.031971 0.09903 rpy=0.053337 0.19165 0.010169
- joint finger22: limit lower=0.011072 upper=1.687426 effort=0 velocity=0 -> lower=0.011072 upper=1.265777 effort=0 velocity=0; mimic joint=finger21 multiplier=0.9206 offset=0.011072 -> joint=finger21 multiplier=1.141100 offset=0.011072
- joint finger23: limit lower=0.011072 upper=1.687426 effort=0 velocity=0 -> lower=0 upper=1.57 effort=0 velocity=0
- joint finger31: limit lower=0 upper=1.396263 effort=0 velocity=0 -> lower=0.000000 upper=1.099557 effort=0 velocity=0; origin xyz=-0.013501 -0.0105 0.10286 rpy=0 0.10214 0 -> xyz=-0.013501 -0.0105 0.10186 rpy=0 0.21461 0
- joint finger32: limit lower=0.011072 upper=1.687426 effort=0 velocity=0 -> lower=0.011072 upper=1.265777 effort=0 velocity=0; mimic joint=finger31 multiplier=0.9206 offset=0.011072 -> joint=finger31 multiplier=1.141100 offset=0.011072
- joint finger33: limit lower=0 upper=1.396263 effort=0 velocity=0 -> lower=0 upper=1.57 effort=0 velocity=0; origin xyz=0 0 0 rpy=0 0 0 -> xyz=-0.00755240178743652 0 -0.00366555552280307 rpy=-3.02514163263918 0 -1.5707963267949
- joint finger41: limit lower=0 upper=1.396263 effort=0 velocity=0 -> lower=0.000000 upper=1.082104 effort=0 velocity=0; origin xyz=-0.015081 0.010971 0.10183 rpy=-0.052889 0.14148 -0.0074648 -> xyz=-0.015081 0.010971 0.10083 rpy=-0.053755 0.22825 -0.012175
- joint finger42: limit lower=0.011072 upper=1.687426 effort=0 velocity=0 -> lower=0.011072 upper=1.242074 effort=0 velocity=0; mimic joint=finger41 multiplier=0.9206 offset=0.011072 -> joint=finger41 multiplier=1.137600 offset=0.011072
- joint finger43: limit lower=0 upper=1.396263 effort=0 velocity=0 -> lower=0 upper=1.57 effort=0 velocity=0
- joint finger51: limit lower=0 upper=1.396263 effort=0 velocity=0 -> lower=0.000000 upper=1.151917 effort=0 velocity=0; origin xyz=-0.013081 0.032156 0.097798 rpy=-0.078754 0.073706 -0.0058113 -> xyz=-0.013081 0.032156 0.096798 rpy=-0.080003 0.19132 -0.015244
- joint finger52: limit lower=0.011072 upper=1.687426 effort=0 velocity=0 -> lower=0.011072 upper=1.337620 effort=0 velocity=0; mimic joint=finger51 multiplier=0.9206 offset=0.011072 -> joint=finger51 multiplier=1.151600 offset=0.011072

File: DH116/DH116_URDF_MJCF_Files/DH116-R000-A1/urdf/DH116-R000-A1.urdf (robot description, URDF)
Before this commit: robot DH116-R000-A1, 17 links, 16 joints
Links:
- link base_link: mass 0.10866 -> 0.179403497856359
- link finger11_link: mass 0.010254 -> 0.0100352882231459
- link finger12_link: mass 0.010145 -> 0.0101454287024189
- link finger13_link: mass 0.020548 -> 0.0205479157169511
- link finger14_link: mass 0.00064654 -> 0.000646540582627886
- link finger21_link: mass 0.0067143 -> 0.00671413102935742
- link finger22_link: mass 0.014789 -> 0.0147920191509636
- link finger23_link: mass 0.00083419 -> 0.000834212738824978
- link finger31_link: mass 0.0067141 -> 0.00671424935038803
- link finger32_link: mass 0.017444 -> 0.0174420825086021
- link finger33_link: mass 0.00083416 -> 0.000834213510333441
- link finger41_link: mass 0.006714 -> 0.00671412244916
- link finger42_link: mass 0.014788 -> 0.014787928293369
- link finger43_link: mass 0.0008342 -> 0.000834213969310814
- link finger51_link: mass 0.0067142 -> 0.0067142387189764
- link finger52_link: mass 0.010445 -> 0.01044516195271
- link finger53_link: mass 0.00059177 -> 0.000591753805906821
Joints:
- joint finger11: limit lower=0 upper=1.047198 effort=0 velocity=0 -> lower=0.000000 upper=0.994838 effort=0 velocity=0; origin xyz=0.018 0.021747 0.043279 rpy=-0.087266 0 0 -> xyz=0.0179999999999996 0.0217472482996747 0.0422789195985737 rpy=-0.0789062242 0.0373113117 0.4408056675
- joint finger12: axis 0 -1 0 -> -1 0 0; limit lower=0 upper=0.523599 effort=0 velocity=0 -> lower=0.000000 upper=0.750492 effort=0 velocity=0; origin xyz=0.018876 0.0049375 -0.0056093 rpy=0 0.95149 0.25585 -> xyz=0.018876 0.0049375 -0.0056093 rpy=0.95149 0 1.8266
- joint finger13: axis 0 -1 0 -> -1 0 0; limit lower=0.004592 upper=0.594583 effort=0 velocity=0 -> lower=0.004592 upper=0.930248 effort=0 velocity=0; mimic joint=finger12 multiplier=0.8808 offset=0.004592 -> joint=finger12 multiplier=1.233400 offset=0.004592; origin xyz=0 0 0.045 rpy=0 0 0 -> xyz=0 0 0.045 rpy=0 0 0.10198
- joint finger14: limit lower=0 upper=1.396263 effort=0 velocity=0 -> lower=0 upper=1.57 effort=0 velocity=0
- joint finger21: limit lower=0 upper=1.396263 effort=0 velocity=0 -> lower=0.000000 upper=1.099557 effort=0 velocity=0; origin xyz=-0.011581 0.031971 0.10003 rpy=-0.052657 0.10625 -0.0055894 -> xyz=-0.011581 0.031971 0.09903 rpy=-0.053527 0.20908 -0.01112
- joint finger22: limit lower=0.011072 upper=1.687426 effort=0 velocity=0 -> lower=0.011072 upper=1.265777 effort=0 velocity=0; mimic joint=finger21 multiplier=0.9206 offset=0.011072 -> joint=finger21 multiplier=1.141100 offset=0.011072
- joint finger23: limit lower=0.011072 upper=1.687426 effort=0 velocity=0 -> lower=0 upper=1.57 effort=0 velocity=0
- joint finger31: limit lower=0 upper=1.396263 effort=0 velocity=0 -> lower=0.000000 upper=1.099557 effort=0 velocity=0; origin xyz=-0.013501 0.0105 0.10286 rpy=0 0.10214 0 -> xyz=-0.013501 0.0105 0.10186 rpy=0 0.22857 0
- joint finger32: limit lower=0.011072 upper=1.687426 effort=0 velocity=0 -> lower=0.011072 upper=1.265777 effort=0 velocity=0; mimic joint=finger31 multiplier=0.9206 offset=0.011072 -> joint=finger31 multiplier=1.141100 offset=0.011072
- joint finger33: limit lower=0 upper=1.396263 effort=0 velocity=0 -> lower=0 upper=1.57 effort=0 velocity=0
- joint finger41: limit lower=0 upper=1.396263 effort=0 velocity=0 -> lower=0.000000 upper=1.082104 effort=0 velocity=0; origin xyz=-0.015081 -0.010971 0.10183 rpy=0.052889 0.14148 0.0074648 -> xyz=-0.015081 -0.010971 0.10083 rpy=0.053587 0.21431 0.011407
- joint finger42: limit lower=0.011072 upper=1.687426 effort=0 velocity=0 -> lower=0.011072 upper=1.242074 effort=0 velocity=0; mimic joint=finger41 multiplier=0.9206 offset=0.011072 -> joint=finger41 multiplier=1.137600 offset=0.011072
- joint finger43: limit lower=0 upper=1.396263 effort=0 velocity=0 -> lower=0 upper=1.57 effort=0 velocity=0
- joint finger51: limit lower=0 upper=1.396263 effort=0 velocity=0 -> lower=0.000000 upper=1.151917 effort=0 velocity=0; origin xyz=-0.013081 -0.032156 0.097798 rpy=0.078754 0.073706 0.0058113 -> xyz=-0.013081 -0.032156 0.096798 rpy=0.08007 0.19563 0.015596
- joint finger52: limit lower=0.011072 upper=1.687426 effort=0 velocity=0 -> lower=0.011072 upper=1.337620 effort=0 velocity=0; mimic joint=finger51 multiplier=0.9206 offset=0.011072 -> joint=finger51 multiplier=1.151600 offset=0.011072
